File: TAPRX-888 KiCad - Copy/TAPRX-888.kicad_sch (KiCad schematic)
At the start: 126 parts, among them J1 CONN_SMA_JACK_EDGE_JLC_With_N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, J11 Conn_JTAG10-mini, J2 CONN_SMA_JACK_EDGE_JLC_With_N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, J3 CONN_SMA_JACK_EDGE_JLC_With_N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, J4 CONN_SMA_JACK_EDGE_JLC_With_N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, J5 USB-3.0, U1 AP2114H-3.3TRG1, U10 XO-19.2MHZ, U11 CYUSB3014-BZXCT, U2 AP2114H-3.3TRG1, U3 AP2114H-3.3TRG1, U4 LP5907MFX-3.3, U5 UMW AMS1117-1.2, U6 AD8370, U7 TVS-SP3011, U8 LTC2208CUP#PBF, U9 MX25L3233FM2I

Commit message: proper update
Parts:
- removed J1, J2, J3, J4: CONN_SMA_JACK_EDGE_JLC_With_Nut, TIS_Footprints:SMA_Jack_EdgeMount_JLC_With_Nut, symbol TIS:CONN_SMA_JACK_EDGE_JLC_with_nut
- added J1, J2, J3, J4: CONN_SMA_JACK_RA, TIS_Footprints:SMA-RA-Jack, symbol Library:CONN_SMA_JACK_RA
- H1, H2, H3, H4, TP20: now in the parts list
Connections:
- net Clock/EXT_REF_IN: now also J1.1 (In)
- net Front_End_Filter/RF_ATTEN__IN: now also J3.1 (In)
- net Front_End_Filter/RF_IN: now also J2.1 (In)
- net GND: now also J1.2 (Ext), J2.2 (Ext), J3.2 (Ext), J4.2 (Ext)
- net at TP1.1: now also J4.1 (In)
- net at C27.2, R3.2, R5.1: no longer C31.1
- net at C26.2, R2.1, R4.1: no longer C30.1
- net at R4.2, U8.8 (AIN+): now also C30.1
- net at R5.2, U8.9 (AIN-): now also C31.1
Other:
- moved on the sheet: C30, C31, R2, R3, R4, R5
