File: TAPRX-888.kicad_pcb (KiCad board)
At the start: 6 copper layers, 83.5 x 99.4 mm, 225 parts, among them J1 CONN_SMA_JACK_EDGE_JLC_With_N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, J10 U.FL-R, J11 Conn_JTAG10-mini, J2 CONN_SMA_JACK_EDGE_JLC_With_N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, J3 CONN_SMA_JACK_EDGE_JLC_With_N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, J4 CONN_SMA_JACK_EDGE_JLC_With_N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, J5 USB-3.0, J6 Conn_01x03, J7 Conn_01x03, J8 Conn_01x03, J9 Conn_01x03, Q1 PMOS Si2343DS, Q2 MMBT3904, Q3 PMOS Si2343DS, U1 AP2114H-3.3TRG1, U10 XO-19.2MHZ, U11 CYUSB3014-BZXCT, U14 LP5907MFX-3.3, U16 TLV3501, U18 NC7SV157, U19 74LVC2G14, U2 AP2114H-3.3TRG1, U20 Si5351A, U21 NC7SV157, U22 SN65LVDS1, U3 AP2114H-3.3TRG1, U4 LP5907MFX-3.3, U5 UMW AMS1117-1.2, U6 AD8370, U7 TVS-SP3011, U8 LTC2208CUP#PBF, U9 MX25L3233FM2I, X1 TCXO-27M

Commit message: refdes and silk cleanup, now produces a zero ERC/DRC error, zero DRC warning output
Parts:
- moved C2 0.10 mm to (149.9, 87.0)
Changed lines of the file:
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@@
 		(tags "capacitor 0603")
 		(property "Reference" "R61"
-			(at 0 -1.25 90)
+			(at -0.1 -1.35 90)
 			(unlocked yes)
 			(layer "F.SilkS")
@@
 		(at 156 81)
 		(property "Reference" "U11"
-			(at -4.1 -6.2 0)
+			(at 6.3 4.3 90)
 			(unlocked yes)
 			(layer "F.SilkS")
@@
 		(duplicate_pad_numbers_are_jumpers no)
 		(fp_line
-			(start -5.5 -4.39)
-			(end -5.5 -3.01)
+			(start -5.4 -5.4)
+			(end -3.1 -5.4)
 			(stroke
 				(width 0.12)
@@
 		)
 		(fp_line
-			(start -5.5 5.5)
-			(end -5.5 3)
+			(start -5.4 -3.1)
+			(end -5.4 -5.4)
 			(stroke
 				(width 0.12)
@@
 		)
 		(fp_line
-			(start -3 -5.51)
-			(end -4.38 -5.51)
+			(start -5.4 5.4)
+			(end -5.4 3)
 			(stroke
 				(width 0.12)
@@
 		)
 		(fp_line
-			(start -3 5.5)
-			(end -5.5 5.5)
+			(start -3 5.4)
+			(end -5.4 5.4)
 			(stroke
 				(width 0.12)
@@
 		)
 		(fp_line
-			(start 3 -5.5)
-			(end 5.5 -5.5)
+			(start 3 5.4)
+			(end 5.4 5.4)
 			(stroke
 				(width 0.12)
@@
 		)
 		(fp_line
-			(start 3 5.5)
-			(end 5.5 5.5)
+			(start 3.1 -5.4)
+			(end 5.4 -5.4)
 			(stroke
 				(width 0.12)
@@
 		)
 		(fp_line
-			(start 5.5 -5.5)
-			(end 5.5 -3)
+			(start 5.4 -5.4)
+			(end 5.4 -3.1)
 			(stroke
 				(width 0.12)
@@
 		)
 		(fp_line
-			(start 5.5 5.5)
-			(end 5.5 3)
+			(start 5.4 5.4)
+			(end 5.4 2.9)
 			(stroke
 				(width 0.12)
@@
 		)
 		(fp_circle
-			(center -5.5 -5.5)
-			(end -5.5 -5.4)
+			(center -4.4 -5.9)
+			(end -4.4 -5.8)
 			(stroke
 				(width 0.2)
@@
 		(tags "capacitor 0603")
 		(property "Reference" "R20"
-			(at 1.8 0.95 0)
+			(at 1.9 -3.8 90)
 			(unlocked yes)
 			(layer "F.SilkS")
@@
 	(footprint "Library:C_0603"
 		(layer "F.Cu")
-		(at 150 87)
+		(at 149.9 87)
 		(descr "Capacitor SMD 0603, reflow soldering, AVX (see smccp.pdf)")
 		(tags "capacitor 0603")
 		(property "Reference" "C2"
-			(at -1.9 0 90)
+			(at 0 1.4 0)
 			(unlocked yes)
 			(layer "F.SilkS")
@@
 		(tags "capacitor 0603")
 		(property "Reference" "C77"
-			(at -1.65 -1 0)
+			(at -1.15 2.3 90)
 			(unlocked yes)
 			(layer "F.SilkS")
@@
 		(at 156 95)
 		(property "Reference" "U8"
-			(at 0 -6.1 0)
+			(at 5.7 3.4 90)
 			(unlocked yes)
 			(layer "F.SilkS")
-			(hide yes)
 			(effects
 				(font
-					(size 0.75 0.75)
-					(thickness 0.1)
+					(size 0.8 0.8)
+					(thickness 0.15)
 				)
 			)
@@
 		)
 		(fp_text user "REF**"
-			(at 5.9 3.4 90)
-			(layer "F.SilkS")
-			(effects
-				(font
-					(size 0.8 0.8)
-					(thickness 0.15)
-				)
-			)
-		)
-		(fp_text user "REF**"
 			(at -0.1524 -7.5692 0)
 			(layer "F.Fab")
@@
 	)
 	(gr_line
-		(start 158.2 101.7)
-		(end 158.8 102.2)
+		(start 144.2 86.3)
+		(end 145.2 85.7)
+		(stroke
+			(width 0.15)
+			(type solid)
+		)
+		(layer "F.SilkS")
+	)
+	(gr_line
+		(start 144.2 87.4)
+		(end 144.2 86.3)
+		(stroke
+			(width 0.15)
+			(type solid)
+		)
+		(layer "F.SilkS")
+	)
+	(gr_line
+		(start 148.3 86.1)
+		(end 148.5 85.7)
+		(stroke
+			(width 0.15)
+			(type solid)
+		)
+		(layer "F.SilkS")
+	)
+	(gr_line
+		(start 158.1 101.65)
+		(end 158.7 102.15)
 		(stroke
 			(width 0.15)

Commit message: initial USB2/3 tweaks
Parts:
- U12, U13, U15, U17: value ~ -> BAV99
- moved C39 0.70 mm to (157.3, 74.0)
- moved C40 0.10 mm to (156.1, 74.0)
Connections:
- net Net-(U11-SSTXM) renamed /FX3_SSTX-
- net Net-(U11-SSTXP) renamed /FX3_SSTX+
Routing:
- net /ID6: track 34.1 -> 39.7 mm
- net /FX3_SSTX-: track 3.84 -> 2.79 mm
