File: refclk.kicad_sch (KiCad schematic)
At the start: 57 parts, among them J10 U.FL-R, Q1 PMOS Si2343DS, Q2 MMBT3904, Q3 PMOS Si2343DS, U14 LP5907MFX-3.3, U15 BAV99, U16 TLV3501, U17 BAV99, U18 NC7SV157, U19 74LVC2G14, U20 Si5351A, U21 NC7SV157, U22 SN65LVDS1, X1 TCXO-27M

Commit message: clean baked-in field junk; strip footprint LCSC; sync board
- board + schematic: clear Datasheet fields holding stray LCSC numbers,
  fix U8 doubled #PBF MPN
- library footprints: empty baked-in LCSC Part # (authoritative on the
  schematic; blocks Update-Footprints from clobbering board part numbers)
- Update PCB from Schematic sync (U8 LCSC, TP exclude-from-pos)
ERC clean; DRC clean with schematic parity.
Parts:
- X1: Comment alternate: C46598427 ±2ppm -> (none)
Changed lines of the file:
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@@
 		(in_bom no)
 		(on_board yes)
-		(in_pos_files yes)
+		(in_pos_files no)
 		(dnp no)
 		(property "Reference" "TP17"
@@
 			)
 		)
-		(property "Comment" "alternate: C46598427  ±2ppm"
+		(property "Comment" ""
 			(at 152.654 49.022 0)
 			(hide yes)
@@
 			)
 		)
-		(property "Datasheet" "C25804"
+		(property "Datasheet" ""
 			(at 172.72 120.65 0)
 			(hide yes)
@@
 			)
 		)
-		(property "Datasheet" "C14663"
+		(property "Datasheet" ""
 			(at 191.77 78.74 0)
 			(hide yes)
@@
 			)
 		)
-		(property "Datasheet" "C14663"
+		(property "Datasheet" ""
 			(at 208.28 140.97 0)
 			(hide yes)
@@
 			)
 		)
-		(property "Datasheet" "C14663"
+		(property "Datasheet" ""
 			(at 243.84 48.26 0)
 			(hide yes)
@@
 			)
 		)
-		(property "Datasheet" "C25804"
+		(property "Datasheet" ""
 			(at 231.14 156.21 0)
 			(hide yes)
@@
 			)
 		)
-		(property "Datasheet" "C14663"
+		(property "Datasheet" ""
 			(at 256.54 143.51 0)
 			(hide yes)
@@
 		(in_bom no)
 		(on_board yes)
-		(in_pos_files yes)
+		(in_pos_files no)
 		(dnp no)
 		(property "Reference" "TP15"
@@
 			)
 		)
-		(property "Datasheet" "C14663"
+		(property "Datasheet" ""
 			(at 132.08 133.35 0)
 			(hide yes)
@@
 		(in_bom no)
 		(on_board yes)
-		(in_pos_files yes)
+		(in_pos_files no)
 		(dnp no)
 		(property "Reference" "TP16"
@@
 			)
 		)
-		(property "Datasheet" "C25804"
+		(property "Datasheet" ""
 			(at 78.74 76.2 0)
 			(hide yes)
@@
 			)
 		)
-		(property "Datasheet" "C22935"
+		(property "Datasheet" ""
 			(at 151.13 139.7 0)
 			(hide yes)
@@
 			)
 		)
-		(property "Datasheet" "C25804"
+		(property "Datasheet" ""
 			(at 78.74 60.96 0)
 			(hide yes)
@@
 		(in_bom no)
 		(on_board yes)
-		(in_pos_files yes)
+		(in_pos_files no)
 		(dnp no)
 		(property "Reference" "TP19"
@@
 			)
 		)
-		(property "Datasheet" "C25804"
+		(property "Datasheet" ""
 			(at 158.75 133.35 0)
 			(hide yes)
@@
 			)
 		)
-		(property "Datasheet" "C22935"
+		(property "Datasheet" ""
 			(at 63.5 80.01 0)
 			(hide yes)
@@
 			)
 		)
-		(property "Datasheet" "C14663"
+		(property "Datasheet" ""
 			(at 87.63 72.39 0)
 			(hide yes)
@@
 			)
 		)
-		(property "Datasheet" "C23138"
+		(property "Datasheet" ""
 			(at 88.9 101.6 0)
 			(hide yes)
@@
 			)
 		)
-		(property "Datasheet" "C14663"
+		(property "Datasheet" ""
 			(at 95.25 111.76 0)
 			(hide yes)
@@
 			)
 		)
-		(property "Datasheet" "C25804"
+		(property "Datasheet" ""
 			(at 63.5 36.83 0)
 			(hide yes)
@@
 			)
 		)
-		(property "Datasheet" "C14663"
+		(property "Datasheet" ""
 			(at 54.61 101.6 0)
 			(hide yes)
@@
 			)
 		)
-		(property "Datasheet" "C23138"
+		(property "Datasheet" ""
 			(at 73.66 101.6 0)
 			(hide yes)
@@
 		(in_bom no)
 		(on_board yes)
-		(in_pos_files yes)
+		(in_pos_files no)
 		(dnp no)
 		(property "Reference" "TP18"
@@
 			)
 		)
-		(property "Datasheet" "C22935"
+		(property "Datasheet" ""
 			(at 95.25 86.36 0)
 			(hide yes)
@@
 			)
 		)
-		(property "Datasheet" "C14663"
+		(property "Datasheet" ""
 			(at 184.15 144.78 0)
 			(hide yes)
