File: TAPRX-888.kicad_sch (KiCad schematic)
At the start: 126 parts, among them J1 CONN_SMA_JACK_EDGE_JLC_With_N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, J11 Conn_JTAG10-mini, J2 CONN_SMA_JACK_EDGE_JLC_With_N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, J3 CONN_SMA_JACK_EDGE_JLC_With_N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, J4 CONN_SMA_JACK_EDGE_JLC_With_N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, J5 USB-3.0, U1 AP2114H-3.3TRG1, U10 XO-19.2MHZ, U11 CYUSB3014-BZXCT, U2 AP2114H-3.3TRG1, U3 AP2114H-3.3TRG1, U4 LP5907MFX-3.3, U5 UMW AMS1117-1.2, U6 AD8370, U7 TVS-SP3011, U8 LTC2208CUP#PBF, U9 MX25L3233FM2I

Commit message: clean baked-in field junk; strip footprint LCSC; sync board
- board + schematic: clear Datasheet fields holding stray LCSC numbers,
  fix U8 doubled #PBF MPN
- library footprints: empty baked-in LCSC Part # (authoritative on the
  schematic; blocks Update-Footprints from clobbering board part numbers)
- Update PCB from Schematic sync (U8 LCSC, TP exclude-from-pos)
ERC clean; DRC clean with schematic parity.
Parts:
- J3, R22: now in the parts list
Changed lines of the file:
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@@
 		(in_bom no)
 		(on_board yes)
-		(in_pos_files yes)
+		(in_pos_files no)
 		(dnp no)
 		(property "Reference" "TP20"
@@
 		(body_style 1)
 		(exclude_from_sim no)
-		(in_bom no)
+		(in_bom yes)
 		(on_board yes)
-		(in_pos_files no)
+		(in_pos_files yes)
 		(dnp yes)
 		(fields_autoplaced yes)
@@
 		(in_bom no)
 		(on_board yes)
-		(in_pos_files yes)
+		(in_pos_files no)
 		(dnp no)
 		(property "Reference" "TP10"
@@
 		(in_bom no)
 		(on_board yes)
-		(in_pos_files yes)
+		(in_pos_files no)
 		(dnp no)
 		(property "Reference" "TP21"
@@
 		(in_bom no)
 		(on_board yes)
-		(in_pos_files yes)
+		(in_pos_files no)
 		(dnp no)
 		(fields_autoplaced yes)
@@
 		(in_bom no)
 		(on_board yes)
-		(in_pos_files yes)
+		(in_pos_files no)
 		(dnp no)
 		(property "Reference" "TP13"
@@
 		(in_bom no)
 		(on_board yes)
-		(in_pos_files yes)
+		(in_pos_files no)
 		(dnp no)
 		(fields_autoplaced yes)
@@
 		(in_bom no)
 		(on_board yes)
-		(in_pos_files yes)
+		(in_pos_files no)
 		(dnp no)
 		(fields_autoplaced yes)
@@
 		(in_bom no)
 		(on_board yes)
-		(in_pos_files yes)
+		(in_pos_files no)
 		(dnp no)
 		(property "Reference" "TP11"
@@
 		(in_bom no)
 		(on_board yes)
-		(in_pos_files yes)
+		(in_pos_files no)
 		(dnp no)
 		(fields_autoplaced yes)
@@
 		(in_bom no)
 		(on_board yes)
-		(in_pos_files yes)
+		(in_pos_files no)
 		(dnp no)
 		(fields_autoplaced yes)
@@
 		(in_bom no)
 		(on_board yes)
-		(in_pos_files yes)
+		(in_pos_files no)
 		(dnp no)
 		(property "Reference" "TP14"
@@
 		(in_bom no)
 		(on_board yes)
-		(in_pos_files yes)
+		(in_pos_files no)
 		(dnp no)
 		(fields_autoplaced yes)
@@
 		(body_style 1)
 		(exclude_from_sim no)
-		(in_bom no)
+		(in_bom yes)
 		(on_board yes)
 		(in_pos_files yes)
@@
 		(in_bom no)
 		(on_board yes)
-		(in_pos_files yes)
+		(in_pos_files no)
 		(dnp no)
 		(fields_autoplaced yes)
@@
 		(in_bom no)
 		(on_board yes)
-		(in_pos_files yes)
+		(in_pos_files no)
 		(dnp no)
 		(property "Reference" "TP12"
@@
 		(in_bom no)
 		(on_board yes)
-		(in_pos_files yes)
+		(in_pos_files no)
 		(dnp no)
 		(property "Reference" "TP3"
@@
 		(in_bom no)
 		(on_board yes)
-		(in_pos_files yes)
+		(in_pos_files no)
 		(dnp no)
 		(property "Reference" "TP9"

Commit message: Q1/Q3 D/S swap, TP11, TP12 to TPTiny and relocate
Parts:
- TP11, TP12: footprint Library:TP -> Library:TP-Tiny
Changed lines of the file:
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@@
 			)
 		)
-		(property "Footprint" "Library:TP"
+		(property "Footprint" "Library:TP-Tiny"
 			(at 275.59 107.95 0)
 			(hide yes)
@@
 			)
 		)
-		(property "Footprint" "Library:TP"
+		(property "Footprint" "Library:TP-Tiny"
 			(at 275.59 110.49 0)
 			(hide yes)
