File: _restore_backup_2026-08-16T11-04-01-585/TAPRX-888.kicad_pcb (KiCad board)
At the start: 6 copper layers, 83.5 x 99.4 mm, 225 parts, among them J1 CONN_SMA_JACK_EDGE_JLC_With_N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, J10 U.FL-R, J11 Conn_JTAG10-mini, J2 CONN_SMA_JACK_EDGE_JLC_With_N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, J3 CONN_SMA_JACK_EDGE_JLC_With_N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, J4 CONN_SMA_JACK_EDGE_JLC_With_N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, J5 USB-3.0, J6 Conn_01x03, J7 Conn_01x03, J8 Conn_01x03, J9 Conn_01x03, Q1 PMOS Si2343DS, Q2 MMBT3904, Q3 PMOS Si2343DS, U1 AP2114H-3.3TRG1, U10 XO-19.2MHZ, U11 CYUSB3014-BZXCT, U12 BAV99, U13 BAV99, U14 LP5907MFX-3.3, U15 BAV99, U16 TLV3501, U17 BAV99, U18 NC7SV157, U19 74LVC2G14, U2 AP2114H-3.3TRG1, U20 Si5351A, U21 NC7SV157, U22 SN65LVDS1, U3 AP2114H-3.3TRG1, U4 LP5907MFX-3.3, U5 UMW AMS1117-1.2, U6 AD8370, U7 TVS-SP3011, U8 LTC2208CUP#PBF, U9 MX25L3233FM2I, X1 TCXO-27M

Commit message: USB2/3 tweaks pt.2
Connections:
- J5 pad 8: /SSRX+ -> /SSRX-
- J5 pad 9: /SSRX- -> /SSRX+
- U7 pad 1: /SSRX- -> /SSRX+
- U7 pad 13: /SSRX+ -> /SSRX-
- U7 pad 14: /SSRX- -> /SSRX+
- U7 pad 2: /SSRX+ -> /SSRX-
Routing:
- net /ID2: track 21.0 -> 22.5 mm
- net /SSTX+: track 12.0 -> 10.9 mm, vias 1 -> 0
- net /SSTX-: track 12.3 -> 11.4 mm, vias 1 -> 0
- net /SSRX-: track 15.6 -> 14.7 mm, vias 1 -> 0
- net /SSRX+: track 15.4 -> 15.3 mm, vias 1 -> 2
