File: _restore_backup_2026-08-16T11-04-01-585/TAPRX-888.kicad_sch (KiCad schematic)
At the start: 126 parts, among them J1 CONN_SMA_JACK_EDGE_JLC_With_N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, J11 Conn_JTAG10-mini, J2 CONN_SMA_JACK_EDGE_JLC_With_N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, J3 CONN_SMA_JACK_EDGE_JLC_With_N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, J4 CONN_SMA_JACK_EDGE_JLC_With_N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, J5 USB-3.0, U1 AP2114H-3.3TRG1, U10 XO-19.2MHZ, U11 CYUSB3014-BZXCT, U2 AP2114H-3.3TRG1, U3 AP2114H-3.3TRG1, U4 LP5907MFX-3.3, U5 UMW AMS1117-1.2, U6 AD8370, U7 TVS-SP3011, U8 LTC2208CUP#PBF, U9 MX25L3233FM2I

Commit message: USB2/3 tweaks pt.2
Connections:
- net SSRX+: no longer J5.8 (SSRX-), U7.2
- net SSRX-: now also J5.8 (SSRX-), U7.2
Changed lines of the file:
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@@
 		)
 	)
-	(label "SSRX+"
+	(label "SSRX-"
 		(at 182.88 208.28 0)
 		(fields_autoplaced yes)
