File: mechanical/endplate-rear/endplate-rear.kicad_pcb (KiCad board)
At the start: 2 copper layers, 88 x 38 mm, 0 parts

Commit message: update design and fab notes text on PCB drawings
Other:
- board text added: "DESIGN NOTES ======================================== Outline 88x38mm R4.5mm; M3 corner holes Ø3.4mm USB 3.0 opening 12.5x12.9mm, STATUS hole Ø2.0mm to view the D3 LED (body-center aligned via fit-check. Shield: F+B copper pour, perimeter 0.3/0.6mm via stitch, Ø7mm exposed-copper mask at each M3 (screw grounds to enclosure). Via/keepout/mask exposure was script-generated (scripts/stitch_perimeter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"
- board text added: "FABRICATION SPECIFICATION ======================================== Project: TAPRX-888 Rear End Plate GENERAL Layers: 2 Material: FR4, standard Tg Finished Thickness: 1.6mm (~63 mil) +/-10% Surface Finish: ENIG Solder Mask: Blue, both sides Silkscreen: White, both sides IPC Class: 2 STACKUP F.Cu 1 oz (0.035mm) core 1.51mm FR4 (Er 4.5) B.Cu 1 oz (0.035mm) (1.6mm nominal, ENIG) CONTROLLED IMPEDANCE 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"
- board text removed: "REAR PLATE (USB). X-mirrored vs front (outside view). Enclosure end plate; F+B GND shield, chassis-grounded via M3 screws. No active parts. Outline 88x38 R4.5; M3 corner holes Ø3.4 @ +/-41,+/-14.21 (plate screws on, full face). USB 3.0 opening 12.5x12.9 centered at plate (25.04, 15.49). STATUS hole Ø2.0 at plate (44.0, 9.51) to view the D3 LED (body-center aligned via the fit-check; D3 3D model +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"
Changed lines of the file:
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@@
 		)
 	)
-	(gr_text "REAR PLATE (USB). X-mirrored vs front (outside view). Enclosure end plate; F+B GND shield, chassis-grounded via M3 screws. No active parts.\nOutline 88x38 R4.5; M3 corner holes Ø3.4 @ +/-41,+/-14.21 (plate screws on, full face).\nUSB 3.0 opening 12.5x12.9 centered at plate (25.04, 15.49).\nSTATUS hole Ø2.0 at plate (44.0, 9.51) to view the D3 LED (body-center aligned via the fit-check; D3 3D model +0.5 Z).\nShield: F+B GND pour, perimeter 0.3/0.6 via stitch, Ø7 exposed-copper mask at each M3 (screw grounds to enclosure). Script-generated (scripts/stitch_perimeter.py) -- do not hand-edit.\nplate Y from floor edge Y=0, +Y = up. Dimensions dialed in against the 3D fit-check; open in KiCad 10 to confirm."
-		(at 148.59 133.35 0)
+	(gr_text "DESIGN NOTES\n========================================\n\nOutline 88x38mm R4.5mm; M3 corner holes Ø3.4mm\nUSB 3.0 opening 12.5x12.9mm, STATUS hole Ø2.0mm to view the D3 LED (body-center aligned via fit-check.\nShield: F+B copper pour, perimeter 0.3/0.6mm via stitch,\n Ø7mm exposed-copper mask at each M3 (screw grounds to enclosure). \n Via/keepout/mask exposure was script-generated (scripts/stitch_perimeter.py)"
+		(at 17.5 35 0)
 		(layer "Cmts.User")
 		(effects
 			(font
-				(size 1 1)
-				(thickness 0.15)
+				(size 1.5 1.5)
+				(thickness 0.3)
+				(bold yes)
 			)
+			(justify left)
 		)
 	)
+	(gr_text "FABRICATION SPECIFICATION\n========================================\nProject: TAPRX-888 Rear End Plate\n\nGENERAL\n  Layers:             2\n  Material:           FR4, standard Tg\n  Finished Thickness: 1.6mm (~63 mil) +/-10%\n  Surface Finish:     ENIG\n  Solder Mask:        Blue, both sides\n  Silkscreen:         White, both sides\n  IPC Class:          2\n\nSTACKUP\n  F.Cu     1 oz  (0.035mm)\n  core     1.51mm  FR4 (Er 4.5)\n  B.Cu     1 oz  (0.035mm)\n  (1.6mm nominal, ENIG)\n\nCONTROLLED IMPEDANCE\n  None -- non-signal shield plate.\n\nMINIMUM FEATURES  (JLCPCB 2-layer, standard)\n  Track width:    0.15mm\n  Track spacing:  0.15mm\n  Via:            0.60mm dia / 0.30mm drill  (GND stitch ring)\n  Annular ring:   0.15mm\n  Hole-to-hole:   0.50mm (diff net) / 0.25mm (same net)\n  Min PTH drill:  0.30mm\n  Copper-to-edge: 0.50mm\n  Silk:           0.15mm min width, 2.0mm text\n\nVIAS\n  Through-hole only -- no blind/buried vias.\n  Via tenting: both sides (stitch vias covered by mask).\n\nNOTES\n  1. All dimensions in mm unless noted.\n  2. Non-signal shield end plate -- no assembly / BOM / CPL.\n  3. Mounting / LED / USB holes are routed Edge.Cuts cutouts (not drilled)."
+		(at 17.5 147.5 0)
+		(layer "Cmts.User")
+		(effects
+			(font
+				(size 1.5 1.5)
+				(thickness 0.3)
+				(bold yes)
+			)
+			(justify left bottom)
+		)
+	)
